File: heating-control.kicad_pcb (KiCad board)
At the start: 2 copper layers, 142.5 x 72.5 mm, 42 parts, among them IC1 AD5721RBRUZ, IC2 PCF8563T_5,518, IC3 VXO7803-500-M-TR, IC4 LM4040DYM3-2.5-TR, IC5 MR44V064BMAZAATL, IC6 AT25DN256-SSHF-B, J1 Conn_01x08_Male, J4 9242-0-00-80-00-00-08-0, J5 9242-0-00-80-00-00-08-0, J7 9242-0-00-80-00-00-08-0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

Commit message: rev1
Parts:
- removed REF**: TSSOP-16-1EP_4.4x5mm_P0.65mm, Package_SO:TSSOP-16-1EP_4.4x5mm_P0.65mm
- added J2: Conn_01x08_Female, Connector_PinHeader_2.54mm:PinHeader_1x08_P2.54mm_Vertical, F.Cu at (25.8, 26.2)
- added LCD1: LCD_128x64, my-stuff.pretty:lcd_test, F.Cu at (13.5, 3.87)
- added Q1: MMBT3906, Package_TO_SOT_SMD:SOT-23, B.Cu at (43.3, 30.1)
- added R5: 10k, Resistor_SMD:R_0603_1608Metric, B.Cu at (44.2, 25.7)
- added R6: 10k, Resistor_SMD:R_0603_1608Metric, B.Cu at (36.5, 29.1)
- added logo1: logo, footprints:logo_me, F.Cu at (64.5, -12.6)
- moved TP3 7.36 mm to (50.7, 13.5)
- moved R1 5.52 mm to (12.0, -1.13), turned to 0 degrees
- moved C10 5.06 mm to (27.9, 0.67)
- moved C2 4.93 mm to (27.9, 2.17)
- moved R3 4.49 mm to (-41.4, -2.35), turned to 90 degrees
- moved C5 3.50 mm to (13.9, 8.32)
- moved C11 3.46 mm to (14.0, 6.44)
- moved IC1 3.34 mm to (21.6, 3.67)
- moved JP1 2.33 mm to (22.5, 11.6)
Connections:
- U1 pad 13: (no net) -> /LCD_LED_ON
- U1 pad 29: (no net) -> /LCD_RESET
- U1 pad 30: (no net) -> /SPI_CS_LCD
- U1 pad 31: (no net) -> /LCD_A0
Routing:
- net /LCD_LED_ON: track 0.00 -> 114.1 mm
- net /SDA: track 47.2 -> 126.8 mm, vias 0 -> 2
- net /SCL: track 54.7 -> 133.9 mm, vias 0 -> 2
- net /SPI_CS_LCD: track 0.00 -> 72.2 mm, vias 0 -> 1
- net /LCD_A0: track 0.00 -> 71.0 mm, vias 0 -> 1
- net /LCD_RESET: track 0.00 -> 68.6 mm, vias 0 -> 1
- net VCC3V3: track 283.5 -> 346.6 mm
- net /SPI_MOSI: track 94.4 -> 148.5 mm, vias 2 -> 5
- net /SPI_CLK: track 94.3 -> 143.5 mm, vias 0 -> 3
- net /SPI_MISO: track 106.9 -> 120.8 mm, vias 0 -> 2
- net /SPI_CS_FLASH: track 72.1 -> 80.4 mm
- net /ENCODER_B: track 126.4 -> 132.6 mm
- net /SPI_CS_AD5721: track 95.3 -> 100.7 mm
- net /ENCODER_A: track 131.6 -> 136.7 mm
- net Net-(Q1-Pad1): track 0.00 -> 5.06 mm
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Other:
- net class VCC3V3: trace_width 0.5 -> 0.3
- board text added: "RX<-"
- board text added: "SCL"
- board text added: "SDA"
- board text added: "TX->"
- board text added: "heating-control"
- board text added: "rev. 1 / 20210219"
- board text removed: "CC_RXin"
- board text removed: "CC_TXout"

Commit message: latest version
Parts:
- added H1: MountingHole, MountingHole:MountingHole_3.2mm_M3_Pad_Via, F.Cu at (-57.5, 30.0)
- added H2: MountingHole, MountingHole:MountingHole_3.2mm_M3_Pad_Via, F.Cu at (-15.0, 30.0)
- added H3: MountingHole, MountingHole:MountingHole_3.2mm_M3_Pad_Via, F.Cu at (55.0, 30.0)
- added H4: MountingHole, MountingHole:MountingHole_3.2mm_M3_Pad_Via, F.Cu at (67.5, 11.7)
- added H5: MountingHole, MountingHole:MountingHole_3.2mm_M3_Pad_Via, F.Cu at (45.0, -25.0)
- added H6: MountingHole, MountingHole:MountingHole_3.2mm_M3_Pad_Via, F.Cu at (-15.0, -25.0)
- R2, R3: value 10k -> ??k
- R4: value 10k -> 0R
- R5, R6: value 10k -> ??R
Other:
- outline, holes or cut-outs redrawn
