File: heating-control.sch (KiCad schematic (older format))
At the start: 41 parts, among them IC1 AD5721RBRUZ, IC2 PCF8563T_5,518, IC3 VXO7803-500-M-TR, IC4 LM4040DYM3-2.5-TR, IC5 MR44V064BMAZAATL, IC6 AT25DN256-SSHF-B, J1 Conn_01x08_Male, J4 9242-0-00-80-00-00-08-0, J5 9242-0-00-80-00-00-08-0, J7 9242-0-00-80-00-00-08-0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

Commit message: rev1
Parts:
- added J2: Conn_01x08_Female, Connector_PinHeader_2.54mm:PinHeader_1x08_P2.54mm_Vertical, symbol Connector:Conn_01x08_Female
- added LCD1: LCD_128x64, my-stuff.pretty:lcd_test, symbol 1my-stuff:LCD_128x64
- added Q1: MMBT3906, Package_TO_SOT_SMD:SOT-23, symbol Transistor_BJT:MMBT3906
- added R5, R6: 10k, Resistor_SMD:R_0603_1608Metric, symbol Device:R
- added logo?: logo, footprints:logo_me, symbol 1my-stuff:logo
- IC1: symbol heating-control-rescue:AD5721RBRUZ-AD5721RBRUZ -> heating-control-rescue:AD5721RBRUZ-AD5721RBRUZ-heating-control-rescue
- IC2: symbol heating-control-rescue:PCF8563T_5,518-PCF8563T_5_518 -> heating-control-rescue:PCF8563T_5,518-PCF8563T_5_518-heating-control-rescue
- IC3: symbol heating-control-rescue:VXO7803-500-M-TR-VXO7803-500-M-TR -> heating-control-rescue:VXO7803-500-M-TR-VXO7803-500-M-TR-heating-control-rescue
- IC4: symbol heating-control-rescue:LM4040DYM3-2.5-TR-LM4040DYM3-2.5-TR -> heating-control-rescue:LM4040DYM3-2.5-TR-LM4040DYM3-2.5-TR-heating-control-rescue
- gave numbers to parts that had none: 4
Connections:
- net GND: now also J2.2 (Pin_2), LCD1.10 (LED-), LCD1.7 (GND)
- net SCL: now also J2.3 (Pin_3)
- net SDA: now also J2.4 (Pin_4)
- net SPI_CLK: now also LCD1.1 (CLK)
- net SPI_MOSI: now also LCD1.2 (MOSI)
- net VCC3V3: now also J2.1 (Pin_1), LCD1.3 (VCC), R5.2
- net LCD_LED_ON: now reaches U1.13 (GPIO15)
- net LCD_LED_ON: now also R6.2
- net LCD_RESET: now reaches U1.29 (GPIO26_AD)
- net LCD_RESET: now also LCD1.5 (/RESET)
- net SPI_CS_LCD: now reaches U1.30 (GPIO27_AD)
- net SPI_CS_LCD: now also LCD1.6 (/CS)
- net LCD_A0: now reaches U1.31 (GPIO28_AD)
- net LCD_A0: now also LCD1.4 (A0)
- new net: LCD1.11 (LED+), Q1.3 (C)
- new net: Q1.1 (B), R6.1
- new net: Q1.2 (E), R5.1
Other:
- moved on the sheet: U2

Commit message: rev1 annotations
Parts:
- gave numbers to parts that had none: 1
Changed lines of the file:
@@
 	8750 6050 8750 5950
 $Comp
-L 1my-stuff:logo logo?
+L 1my-stuff:logo logo1
 U 1 1 605262C5
 P 10800 6800
-F 0 "logo?" H 10825 6846 50  0000 L CNN
+F 0 "logo1" H 10825 6846 50  0000 L CNN
 F 1 "logo" H 10825 6755 50  0000 L CNN
 F 2 "footprints:logo_me" H 10800 6800 50  0001 C CNN

Commit message: latest version
Parts:
- added H1, H2, H3, H4, H5, H6: MountingHole, MountingHole:MountingHole_3.2mm_M3_Pad_Via, symbol Mechanical:MountingHole
- R2, R3: value 10k -> ??k
- R4: value 10k -> 0R
- R5, R6: value 10k -> ??R
Changed lines of the file:
@@
 P 1600 3000
 F 0 "R2" H 1670 3046 50  0000 L CNN
-F 1 "10k" H 1670 2955 50  0000 L CNN
+F 1 "??k" H 1670 2955 50  0000 L CNN
 F 2 "Resistor_SMD:R_0603_1608Metric" V 1530 3000 50  0001 C CNN
 F 3 "~" H 1600 3000 50  0001 C CNN
@@
 P 2050 3000
 F 0 "R3" H 2120 3046 50  0000 L CNN
-F 1 "10k" H 2120 2955 50  0000 L CNN
+F 1 "??k" H 2120 2955 50  0000 L CNN
 F 2 "Resistor_SMD:R_0603_1608Metric" V 1980 3000 50  0001 C CNN
 F 3 "~" H 2050 3000 50  0001 C CNN
@@
 P 9850 1650
 F 0 "R4" H 9920 1696 50  0000 L CNN
-F 1 "10k" H 9920 1605 50  0000 L CNN
+F 1 "0R" H 9920 1605 50  0000 L CNN
 F 2 "Resistor_SMD:R_0603_1608Metric" V 9780 1650 50  0001 C CNN
 F 3 "~" H 9850 1650 50  0001 C CNN
@@
 P 1950 5600
 F 0 "R5" H 2020 5646 50  0000 L CNN
-F 1 "10k" H 2020 5555 50  0000 L CNN
+F 1 "??R" H 2020 5555 50  0000 L CNN
 F 2 "Resistor_SMD:R_0603_1608Metric" V 1880 5600 50  0001 C CNN
 F 3 "~" H 1950 5600 50  0001 C CNN
@@
 P 2400 5050
 F 0 "R6" H 2470 5096 50  0000 L CNN
-F 1 "10k" H 2470 5005 50  0000 L CNN
+F 1 "??R" H 2470 5005 50  0000 L CNN
 F 2 "Resistor_SMD:R_0603_1608Metric" V 2330 5050 50  0001 C CNN
 F 3 "~" H 2400 5050 50  0001 C CNN
@@
 	1    0    0    -1
 $EndComp
+$Comp
+L Mechanical:MountingHole H1
+U 1 1 6031AE8E
+P 12150 500
+F 0 "H1" H 12250 546 50  0000 L CNN
+F 1 "MountingHole" H 12250 455 50  0000 L CNN
+F 2 "MountingHole:MountingHole_3.2mm_M3_Pad_Via" H 12150 500 50  0001 C CNN
+F 3 "~" H 12150 500 50  0001 C CNN
+	1    12150 500
+	1    0    0    -1
+$EndComp
+$Comp
+L Mechanical:MountingHole H3
+U 1 1 603200D1
+P 12200 800
+F 0 "H3" H 12300 846 50  0000 L CNN
+F 1 "MountingHole" H 12300 755 50  0000 L CNN
+F 2 "MountingHole:MountingHole_3.2mm_M3_Pad_Via" H 12200 800 50  0001 C CNN
+F 3 "~" H 12200 800 50  0001 C CNN
+	1    12200 800
+	1    0    0    -1
+$EndComp
+$Comp
+L Mechanical:MountingHole H4
+U 1 1 6032032A
+P 12200 1100
+F 0 "H4" H 12300 1146 50  0000 L CNN
+F 1 "MountingHole" H 12300 1055 50  0000 L CNN
+F 2 "MountingHole:MountingHole_3.2mm_M3_Pad_Via" H 12200 1100 50  0001 C CNN
+F 3 "~" H 12200 1100 50  0001 C CNN
+	1    12200 1100
+	1    0    0    -1
+$EndComp
+$Comp
+L Mechanical:MountingHole H2
+U 1 1 60320486
+P 12150 1350
+F 0 "H2" H 12250 1396 50  0000 L CNN
+F 1 "MountingHole" H 12250 1305 50  0000 L CNN
+F 2 "MountingHole:MountingHole_3.2mm_M3_Pad_Via" H 12150 1350 50  0001 C CNN
+F 3 "~" H 12150 1350 50  0001 C CNN
+	1    12150 1350
+	1    0    0    -1
+$EndComp
+$Comp
+L Mechanical:MountingHole H5
+U 1 1 60320715
+P 12250 1750
+F 0 "H5" H 12350 1796 50  0000 L CNN
+F 1 "MountingHole" H 12350 1705 50  0000 L CNN
+F 2 "MountingHole:MountingHole_3.2mm_M3_Pad_Via" H 12250 1750 50  0001 C CNN
+F 3 "~" H 12250 1750 50  0001 C CNN
+	1    12250 1750
+	1    0    0    -1
+$EndComp
+$Comp
+L Mechanical:MountingHole H6
+U 1 1 6033C3E7
+P 12200 2300
+F 0 "H6" H 12300 2346 50  0000 L CNN
+F 1 "MountingHole" H 12300 2255 50  0000 L CNN
+F 2 "MountingHole:MountingHole_3.2mm_M3_Pad_Via" H 12200 2300 50  0001 C CNN
+F 3 "~" H 12200 2300 50  0001 C CNN
+	1    12200 2300
+	1    0    0    -1
+$EndComp
